Commit message: Added effort value to effort controller

File: src/robot_pkg/urdf/irb120.urdf (robot description, URDF)
Before this commit: robot irb120, 8 links, 7 joints
Joints:
- joint joint_1: limit lower=-2.87979326579 upper=2.87979326579 effort=0 velocity=4.36332312999 -> lower=-2.87979326579 upper=2.87979326579 effort=20 velocity=4.36332312999
- joint joint_2: limit lower=-1.91986217719 upper=1.91986217719 effort=0 velocity=4.36332312999 -> lower=-1.91986217719 upper=1.91986217719 effort=20 velocity=4.36332312999
- joint joint_3: limit lower=-1.91986217719 upper=1.22173047639 effort=0 velocity=4.36332312999 -> lower=-1.91986217719 upper=1.22173047639 effort=20 velocity=4.36332312999
- joint joint_4: limit lower=-2.79252680319 upper=2.79252680319 effort=0 velocity=5.58505360639 -> lower=-2.79252680319 upper=2.79252680319 effort=20 velocity=5.58505360639
- joint joint_5: limit lower=-2.09439510239 upper=2.09439510239 effort=0 velocity=5.58505360639 -> lower=-2.09439510239 upper=2.09439510239 effort=20 velocity=5.58505360639
- joint joint_6: limit lower=-6.981317008 upper=6.981317008 effort=0 velocity=7.33038285839 -> lower=-6.981317008 upper=6.981317008 effort=20 velocity=7.33038285839

Commit message: Updated limits joint 6

File: src/robot_pkg/urdf/irb120.urdf (robot description, URDF)
Before this commit: robot irb120, 8 links, 7 joints
Joints:
- joint joint_6: limit lower=-6.981317008 upper=6.981317008 effort=20 velocity=7.33038285839 -> lower=-3.0 upper=3.0 effort=20 velocity=7.33038285839
